File: project.sch (EAGLE design)
At the start: 14 parts, among them IC2 LM35DZ_LFT1, IC3 MCP3001T-I_SN, IC4 AT89S52-24PU, Y2 ECS-240-18-5PLX-AGN-TR

Commit message: Update the schematic
Parts:
- removed DC: (no value), pinhead:PINHD-1X2
- added CN1: (no value), adafruit:DCBARRELPTH
Connections:
- removed net N$4: IC4.RST, R1.2, S2.COM
- removed net PROGRAM_SS: IC4.P1.2, JP1.4
- new net PROG_RST: IC4.RST, JP1.4, R1.2, S2.COM
- net GND: now also CN1.GND; no longer DC.2
- net VCC: now also CN1.PWR; no longer DC.1
